Commit message: Update seven_dof_arm.xacro
three joints

File: seven_dof_arm.xacro (robot description, xacro)
@@ -1,3 +1,2 @@
-<!-- three joints -->
 <?xml version="1.0"?>
 <robot name="three_dof_arm" xmlns:xacro="http://ros.org/wiki/xacro">
@@ -106,21 +105,4 @@
     <dynamics damping="50" friction="1"/>
   </joint>
-<!-- ELBOW ROLL LINK
-  <link name="elbow_roll_link" >
-    <visual>
-      <origin xyz="-0.015 0.0 -0.0" rpy="0 ${M_PI/2} 0" />
-      <geometry>
-           <cylinder radius="${elbow_roll_width}" length="${elbow_roll_len}"/>
-      </geometry>
-      <material name="Black" />
-    </visual>
-    <collision>
-      <origin xyz="-0.015 0.0 -0.0" rpy="0 ${M_PI/2} 0" />
-      <geometry>
-            <cylinder radius="${elbow_roll_width}" length="${elbow_roll_len}"/>
-      </geometry>
-    </collision>
-	      <xacro:inertial_matrix mass="1"/>
-  </link> -->
   <joint name="elbow_roll_joint" type="fixed">
     <parent link="shoulder_pitch_link"/>
